File: z80comp2.sch (KiCad schematic (older format))
At the start: 27 parts

Commit message: updated the schematic and project symbol library
Parts:
- added C13, C?: 0.1uF, symbol Device:C_Small
- added R5: 4.7k, symbol Device:R
- added R6: 1M, symbol Device:R
- added R7: 9.1k, symbol Device:R
- added SW1: RESET, symbol Switch:SW_Push
- added U10: 74LS05, symbol 74xx:74LS05
- added U8: 74HC14, symbol 74xx:74HC14
- added U9: LM555, symbol Timer:LM555
- gave numbers to parts that had none: 27
Connections:
- net labels added: RST, UCLK
- wire segments 185 -> 207
- no-connect marks 5 -> 6
Other:
- note added: "Power-on reset"

Commit message: UART done
Parts:
- added C9: 0.1uF, symbol Device:C_Small
- added R7: 120R, symbol Device:R
- added unit 5 of U1
- added unit 4 of U1
- gave numbers to parts that had none: 1
- renumbered C7 to C10, C8 to C11, C9 to C12, C10 to C13, C11 to C14, C12 to C15, C1 to C2, C2 to C3, C3 to C4, C13 to C5, C4 to C6, C5 to C7, C6 to C8, R5 to R4, R6 to R5, R7 to R6, R4 to R8, U8 to U1, U9 to U2, U1 to U3, U5 to U4, U10 to U4, U2 to U5, U3 to U6, U4 to U7, U6 to U8, U7 to U9
Connections:
- wire segments 207 -> 215
- no-connect marks 6 -> 8
Other:
- note added: "Delay the UART ~CS~ for a few ns to bring the\ntiming between R/~W~ and ~CS~ within spec\n(this might have been a red herring and not necessary)"
- moved on the sheet: C1, C10, C11, C12, C13, C14, C15, C5, D1, J1, J2, R1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
